File: hardware/pcb/kino-d4-carrier-a0/01_p4.kicad_sch (KiCad schematic)
At the start: 14 parts, among them J100 P4 JP1 - 26 pin IDC, J101 C6 service - 3V3 sense only, J102 3V3 I2C accessory, U100 TCA9517ADGKR

Commit message: feat(hardware): carrier A0.2 release pass - ready for fabrication with manual checks
Release review of the routed A0.2 carrier (A02-RELEASE.md: release matrix,
manual checks before ordering, bring-up tests). Final status: READY FOR
FABRICATION WITH SPECIFIC MANUAL CHECKS.

- USB-C input survives an unprogrammed STUSB4500 (20 V): D1001 SMF22A,
  R1004 10k, PD and load-switch P-FETs AO4409.
- Boost enable: R1204 100k BOOST_ENABLE to SYS_RAW (LTC2955-1 EN is a 2 uA
  source), Q1202 PMV16UN.
- I2C buffer U100 sides swapped (local bus on the TCA9517 A side's hard
  low); R100/R101 2.2k/22k hold EN low with JP1 pin 1 open.
- R105 SYNC_MASTER pull-down; D903 ESD on FN_N; TP1001 removed.
- SYS_RAW battery path as B.Cu and In2 pours with 25 extra vias; 1 oz inner
  copper in the stackup.
- XIAO socket pads get their solder-mask openings (footprint generator bug).
- Three fiducials per face; vias out of and away from pads; U1200 outline and
  pin-1 mark; legend lines and strokes 0.15 mm; silk association pass;
  CARRIER A0.2 / 2026-10 / S/N marking.
- Fab package (fab_a02.py): Gerbers + job file, drill, zip, placement files,
  fab BOM matched to LCSC by part number, hand-fit socket list, fab notes.
- Firmware constants header kino_carrier_a02.h.

DRC 0 / unconnected 0, ERC 0, verify.py --a02 passes.

Co-Authored-By: Claude Opus 5.5 <noreply@anthropic.com>
Parts:
- added R105: 100k, Resistor_SMD:R_0603_1608Metric, symbol KINO_A0:R105
- C100: value 100n 16V -> 100n 50V
- F100: value PTC 100mA - select -> PTC 100mA
- R100: value 10k -> 2.2k; Design note (none) -> With R101: EN 3.0 V with the P4 on; 0.66 V worst case with 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
- R101: value 1M -> 22k
- U100: Design note B side is local. Do not cascade another B-side offset buffe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 -> A side is local: its hard low suits the STUSB4500 (VIL 0.35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
Connections:
- net GND: now also R105.2
- net I2C_SCL: now also U100.2 (SCLA); no longer U100.7 (SCLB)
- net I2C_SDA: now also U100.3 (SDAA); no longer U100.6 (SDAB)
- net P4_SCL: now also U100.7 (SCLB); no longer U100.2 (SCLA)
- net P4_SDA: now also U100.6 (SDAB); no longer U100.3 (SDAA)
- net SYNC_MASTER: now also R105.1
Other:
- moved on the sheet: C100, F100, J102, R104, TP100, TP101, TP102
