File: hardware/pcb/kino-d4-carrier-a0/06_control.kicad_sch (KiCad schematic)
At the start: 13 parts, among them J600 POGO TEST - SENSE ONLY, J601 EXTERNAL FLASH LOGIC, U600 TCA9539PWR, U601 SN74LVC08APWR

Commit message: feat(hardware): carrier A0.2 - expander port 1 in layout order, channel bundle
U600's port 1 GPIOs (pins 13-20) are interchangeable. North- and
south-bound lines sat interleaved, so every line leaving south crossed
one leaving north. circuit.py now maps P1.0-P1.7 to IMU_INT, RTC_INT_N,
SOFT_KILL, CHARGE_STAT_N, POWER_INT_N, FN_N, HAPTIC_EN, COVER_N (the U600
note had pin 20 as P1.3; it is P1.7). Capture, BOM, netlist, ERC (0) and
PDF are regenerated; firmware must follow the new map.

The five south-bound lines and I2C_SCL now run as one bundle between the
camera 1 and 2 sockets: F rows from U600, vias below the camera lanes,
In2 straight down, vias above the SYNC bus. POWER_INT_N's old route
round the channel goes; the CAM1_3V3 and P4_BUS_EN vias step aside.
RTC_INT_N joins R800 and U801 directly once an MB_3V3 via between them
moves. Router: the last links of RTC_INT_N, SOFT_KILL and IMU_INT.
47 -> 42 open; no clearance or short errors; parity clean.

Co-Authored-By: Claude Opus 5.5 <noreply@anthropic.com>
Parts:
- U600: Design note TCA9539 PW pin map verified against TI; address 0x74 candidate. P1.3 (pin 20) reads charger STAT; configure as INPUT only. -> TCA9539 PW pin map verified against TI; address 0x74 candidate. Port 1 (pins 13-20, P1.0-P1.7): IMU_INT, RTC_INT_N, SOFT_KILL, CHARGE_STAT_N, POWER_INT_N, FN_N, HAPTIC_EN, COVER_N; P1.3 (pin 16) reads charger STAT, configure as INPUT only. Order set by the layout: the lines leaving south take pins 13-17 in the order they reach their parts.
Connections:
- net CHARGE_STAT_N: now also U600.16 (IO1_3); no longer U600.20 (IO1_7)
- net COVER_N: now also U600.20 (IO1_7); no longer U600.13 (IO1_0)
- net FN_N: now also U600.18 (IO1_5); no longer U600.16 (IO1_3)
- net IMU_INT: now also U600.13 (IO1_0); no longer U600.17 (IO1_4)
- net POWER_INT_N: now also U600.17 (IO1_4); no longer U600.14 (IO1_1)
- net RTC_INT_N: now also U600.14 (IO1_1); no longer U600.18 (IO1_5)
Changed lines of the file:
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@@
                   (property "Footprint" "Package_SO:TSSOP-24_4.4x7.8mm_P0.65mm" (at 73.66 64.77 0) (effects (font (size 1 1)) (hide yes)))
                   (property "Datasheet" "https://www.ti.com/lit/ds/symlink/tca9539.pdf" (at 73.66 64.77 0) (effects (font (size 1 1)) (hide yes)))
-                  (property "Design note" "TCA9539 PW pin map verified against TI; address 0x74 candidate. P1.3 (pin 20) reads charger STAT; configure as INPUT only." (at 73.66 64.77 0) (effects (font (size 1 1)) (hide yes)))
+                  (property "Design note" "TCA9539 PW pin map verified against TI; address 0x74 candidate. Port 1 (pins 13-20, P1.0-P1.7): IMU_INT, RTC_INT_N, SOFT_KILL, CHARGE_STAT_N, POWER_INT_N, FN_N, HAPTIC_EN, COVER_N; P1.3 (pin 16) reads charger STAT, configure as INPUT only. Order set by the layout: the lines leaving south take pins 13-17 in the order they reach their parts." (at 73.66 64.77 0) (effects (font (size 1 1)) (hide yes)))
                   (pin "1")(pin "2")(pin "3")(pin "4")(pin "5")(pin "6")(pin "7")(pin "8")(pin "9")(pin "10")(pin "11")(pin "12")(pin "13")(pin "14")(pin "15")(pin "16")(pin "17")(pin "18")(pin "19")(pin "20")(pin "21")(pin "22")(pin "23")(pin "24")
                   (instances (project "KINO_D4_Carrier_A0" (path "/3e6ce248-02da-5043-9ed8-b7ca2a49de29/243a2e2e-3f89-5623-a352-a3b314db1d0e" (reference "U600") (unit 1)))))
@@
                     (property "Intersheetrefs" "${INTERSHEET_REFS}" (at 50.8 78.74 0) (effects (font (size 0.8 0.8)) (hide yes))))
 (wire (pts (xy 91.44 50.8) (xy 96.52 50.8)) (stroke (width 0) (type default)))
-(global_label "COVER_N" (shape bidirectional) (at 96.52 50.8 180)
+(global_label "IMU_INT" (shape bidirectional) (at 96.52 50.8 180)
                     (effects (font (size 0.9 0.9)) (justify left))
                     (property "Intersheetrefs" "${INTERSHEET_REFS}" (at 96.52 50.8 180) (effects (font (size 0.8 0.8)) (hide yes))))
 (wire (pts (xy 91.44 53.33999999999999) (xy 96.52 53.33999999999999)) (stroke (width 0) (type default)))
-(global_label "POWER_INT_N" (shape bidirectional) (at 96.52 53.33999999999999 180)
+(global_label "RTC_INT_N" (shape bidirectional) (at 96.52 53.33999999999999 180)
                     (effects (font (size 0.9 0.9)) (justify left))
                     (property "Intersheetrefs" "${INTERSHEET_REFS}" (at 96.52 53.33999999999999 180) (effects (font (size 0.8 0.8)) (hide yes))))
@@
                     (property "Intersheetrefs" "${INTERSHEET_REFS}" (at 96.52 55.879999999999995 180) (effects (font (size 0.8 0.8)) (hide yes))))
 (wire (pts (xy 91.44 58.419999999999995) (xy 96.52 58.419999999999995)) (stroke (width 0) (type default)))
-(global_label "FN_N" (shape bidirectional) (at 96.52 58.419999999999995 180)
+(global_label "CHARGE_STAT_N" (shape bidirectional) (at 96.52 58.419999999999995 180)
                     (effects (font (size 0.9 0.9)) (justify left))
                     (property "Intersheetrefs" "${INTERSHEET_REFS}" (at 96.52 58.419999999999995 180) (effects (font (size 0.8 0.8)) (hide yes))))
 (wire (pts (xy 91.44 60.959999999999994) (xy 96.52 60.959999999999994)) (stroke (width 0) (type default)))
-(global_label "IMU_INT" (shape bidirectional) (at 96.52 60.959999999999994 180)
+(global_label "POWER_INT_N" (shape bidirectional) (at 96.52 60.959999999999994 180)
                     (effects (font (size 0.9 0.9)) (justify left))
                     (property "Intersheetrefs" "${INTERSHEET_REFS}" (at 96.52 60.959999999999994 180) (effects (font (size 0.8 0.8)) (hide yes))))
 (wire (pts (xy 91.44 63.49999999999999) (xy 96.52 63.49999999999999)) (stroke (width 0) (type default)))
-(global_label "RTC_INT_N" (shape bidirectional) (at 96.52 63.49999999999999 180)
+(global_label "FN_N" (shape bidirectional) (at 96.52 63.49999999999999 180)
                     (effects (font (size 0.9 0.9)) (justify left))
                     (property "Intersheetrefs" "${INTERSHEET_REFS}" (at 96.52 63.49999999999999 180) (effects (font (size 0.8 0.8)) (hide yes))))
@@
                     (property "Intersheetrefs" "${INTERSHEET_REFS}" (at 96.52 66.03999999999999 180) (effects (font (size 0.8 0.8)) (hide yes))))
 (wire (pts (xy 91.44 68.58) (xy 96.52 68.58)) (stroke (width 0) (type default)))
-(global_label "CHARGE_STAT_N" (shape bidirectional) (at 96.52 68.58 180)
+(global_label "COVER_N" (shape bidirectional) (at 96.52 68.58 180)
                     (effects (font (size 0.9 0.9)) (justify left))
                     (property "Intersheetrefs" "${INTERSHEET_REFS}" (at 96.52 68.58 180) (effects (font (size 0.8 0.8)) (hide yes))))

Commit message: feat(hardware): carrier A0.2 - power-side opens, power-button corner
- MB_3V3: three router links join the U900 group, R902 and the main rail.
- Gauge (U701): R701 (BIN pull-down) moves beside its pin, and R702 (GPOUT
  pull-up) moves to the board edge.
- PD controller (U1000): R1004 moves above pin 16, PD_VBUS_SENSE loops
  round it, and C1000 moves onto the USB_VBUS run.
- STAT and charge LED: the charger STAT pin has no layout path out of its
  power copper. It is left open, firmware reads the charge state over I2C,
  and the expander STAT input goes. D1301 (charge LED), R1304, R1109 and
  TP1100 leave the design.
- Power LED: R1303 and D1300 move below U1300.
- Power controller (U1300): C1301 moves beside pin 3. PB and EN drop
  through new vias, and EN runs along the bottom edge to Q1202.

DRC: no clearance or short errors, parity clean, ERC 0, 16 open
connections.

Co-Authored-By: Claude Opus 5.5 <noreply@anthropic.com>
Parts:
- U600: Design note TCA9539 PW pin map verified against TI; address 0x74 candidate. Port 1 (pins 13-20, P1.0-P1.7): IMU_INT, RTC_INT_N, SOFT_KILL, CHARGE_STAT_N, POWER_INT_N, FN_N, HAPTIC_EN, COVER_N; P1.3 (pin 16) reads charger STAT, configure as INPUT only. Order set by the layout: the lines leaving south take pins 13-17 in the order they reach their parts. -> TCA9539 PW pin map verified against TI; address 0x74 candidate. Port 1 (pins 13-20, P1.0-P1.7): IMU_INT, RTC_INT_N, SOFT_KILL, unused, POWER_INT_N, FN_N, HAPTIC_EN, COVER_N; P1.3 (pin 16) is not connected (no layout path from the charger on the far side of the board): firmware reads the charge state from the BQ25798 status registers over I2C; configure P1.3 as an input. Order set by the layout: the lines leaving south take pins 13-17 in the order they reach their parts.
Connections:
- net CHARGE_STAT_N: no longer names the net of U600.16 (IO1_3)
- no-connect marks 1 -> 2
Changed lines of the file:
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@@
                   (property "Footprint" "Package_SO:TSSOP-24_4.4x7.8mm_P0.65mm" (at 73.66 64.77 0) (effects (font (size 1 1)) (hide yes)))
                   (property "Datasheet" "https://www.ti.com/lit/ds/symlink/tca9539.pdf" (at 73.66 64.77 0) (effects (font (size 1 1)) (hide yes)))
-                  (property "Design note" "TCA9539 PW pin map verified against TI; address 0x74 candidate. Port 1 (pins 13-20, P1.0-P1.7): IMU_INT, RTC_INT_N, SOFT_KILL, CHARGE_STAT_N, POWER_INT_N, FN_N, HAPTIC_EN, COVER_N; P1.3 (pin 16) reads charger STAT, configure as INPUT only. Order set by the layout: the lines leaving south take pins 13-17 in the order they reach their parts." (at 73.66 64.77 0) (effects (font (size 1 1)) (hide yes)))
+                  (property "Design note" "TCA9539 PW pin map verified against TI; address 0x74 candidate. Port 1 (pins 13-20, P1.0-P1.7): IMU_INT, RTC_INT_N, SOFT_KILL, unused, POWER_INT_N, FN_N, HAPTIC_EN, COVER_N; P1.3 (pin 16) is not connected (no layout path from the charger on the far side of the board): firmware reads the charge state from the BQ25798 status registers over I2C; configure P1.3 as an input. Order set by the layout: the lines leaving south take pins 13-17 in the order they reach their parts." (at 73.66 64.77 0) (effects (font (size 1 1)) (hide yes)))
                   (pin "1")(pin "2")(pin "3")(pin "4")(pin "5")(pin "6")(pin "7")(pin "8")(pin "9")(pin "10")(pin "11")(pin "12")(pin "13")(pin "14")(pin "15")(pin "16")(pin "17")(pin "18")(pin "19")(pin "20")(pin "21")(pin "22")(pin "23")(pin "24")
                   (instances (project "KINO_D4_Carrier_A0" (path "/3e6ce248-02da-5043-9ed8-b7ca2a49de29/243a2e2e-3f89-5623-a352-a3b314db1d0e" (reference "U600") (unit 1)))))
@@
                     (effects (font (size 0.9 0.9)) (justify left))
                     (property "Intersheetrefs" "${INTERSHEET_REFS}" (at 96.52 55.879999999999995 180) (effects (font (size 0.8 0.8)) (hide yes))))
-(wire (pts (xy 91.44 58.419999999999995) (xy 96.52 58.419999999999995)) (stroke (width 0) (type default)))
-(global_label "CHARGE_STAT_N" (shape bidirectional) (at 96.52 58.419999999999995 180)
-                    (effects (font (size 0.9 0.9)) (justify left))
-                    (property "Intersheetrefs" "${INTERSHEET_REFS}" (at 96.52 58.419999999999995 180) (effects (font (size 0.8 0.8)) (hide yes))))
+(no_connect (at 91.44 58.419999999999995))
 (wire (pts (xy 91.44 60.959999999999994) (xy 96.52 60.959999999999994)) (stroke (width 0) (type default)))
 (global_label "POWER_INT_N" (shape bidirectional) (at 96.52 60.959999999999994 180)

Commit message: feat(hardware): carrier A0.2 - enable test pads, boost EN escape
- CAM2-CAM4_EN have no layout path down to the pogo field J600, so J600
  pads 9-11 become unconnected. TP600-TP602 (1.5 mm probe lands) sit
  beside the enable lines at the top of the board instead.
- U1200 (boost) EN leaves its pin through a via in its pocket. The
  MB_3V3 spur to C801 moves north, and the SYS_RAW riser to pin 7
  swings under the package.

DRC: no clearance or short errors, parity clean, ERC 0, 13 open
connections.

Co-Authored-By: Claude Opus 5.5 <noreply@anthropic.com>
Parts:
- added TP600: CAM2_EN, TestPoint:TestPoint_Pad_D1.5mm, symbol KINO_A0:TP600
- added TP601: CAM3_EN, TestPoint:TestPoint_Pad_D1.5mm, symbol KINO_A0:TP601
- added TP602: CAM4_EN, TestPoint:TestPoint_Pad_D1.5mm, symbol KINO_A0:TP602
- J600: Design note 1.5mm ENIG pads, no paste. Pad 1 offset for fixture orientation. Measure enables; do not drive against U601. Rails are sense points, not a power injection connector. -> 1.5mm ENIG pads, no paste. Pad 1 offset for fixture orientation. Measure enables; do not drive against U601. Rails are sense points, not a power injection connector. Pads 9-11 are unconnected: CAM2-CAM4_EN have no layout path down to the field, so they are probed at TP600-TP602 beside their lines at the top of the board.
Connections:
- net CAM2_EN: now also TP600.1 (CAM2_EN); no longer J600.9 (CAM2_EN)
- net CAM3_EN: now also TP601.1 (CAM3_EN); no longer J600.10 (CAM3_EN)
- net CAM4_EN: now also TP602.1 (CAM4_EN); no longer J600.11 (CAM4_EN)
- no-connect marks 2 -> 5
Other:
- moved on the sheet: J601, R605

Commit message: feat(hardware): carrier A0.2 release pass - ready for fabrication with manual checks
Release review of the routed A0.2 carrier (A02-RELEASE.md: release matrix,
manual checks before ordering, bring-up tests). Final status: READY FOR
FABRICATION WITH SPECIFIC MANUAL CHECKS.

- USB-C input survives an unprogrammed STUSB4500 (20 V): D1001 SMF22A,
  R1004 10k, PD and load-switch P-FETs AO4409.
- Boost enable: R1204 100k BOOST_ENABLE to SYS_RAW (LTC2955-1 EN is a 2 uA
  source), Q1202 PMV16UN.
- I2C buffer U100 sides swapped (local bus on the TCA9517 A side's hard
  low); R100/R101 2.2k/22k hold EN low with JP1 pin 1 open.
- R105 SYNC_MASTER pull-down; D903 ESD on FN_N; TP1001 removed.
- SYS_RAW battery path as B.Cu and In2 pours with 25 extra vias; 1 oz inner
  copper in the stackup.
- XIAO socket pads get their solder-mask openings (footprint generator bug).
- Three fiducials per face; vias out of and away from pads; U1200 outline and
  pin-1 mark; legend lines and strokes 0.15 mm; silk association pass;
  CARRIER A0.2 / 2026-10 / S/N marking.
- Fab package (fab_a02.py): Gerbers + job file, drill, zip, placement files,
  fab BOM matched to LCSC by part number, hand-fit socket list, fab notes.
- Firmware constants header kino_carrier_a02.h.

DRC 0 / unconnected 0, ERC 0, verify.py --a02 passes.

Co-Authored-By: Claude Opus 5.5 <noreply@anthropic.com>
Parts:
- C601, C602: value 100n 16V -> 100n 50V
Changed lines of the file:
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@@
                   (in_bom yes) (on_board yes) (dnp no)
                   (property "Reference" "C601" (at 477.52 52.15 0) (effects (font (size 1.27 1.27))))
-                  (property "Value" "100n 16V" (at 477.52 54.65 0) (effects (font (size 1.0 1.0))))
+                  (property "Value" "100n 50V" (at 477.52 54.65 0) (effects (font (size 1.0 1.0))))
                   (property "Footprint" "Capacitor_SMD:C_0603_1608Metric" (at 477.52 64.77 0) (effects (font (size 1 1)) (hide yes)))
                   (property "Datasheet" "https://www.yageogroup.com/component-documentation/download/specsheet/CC0603KRX7R9BB104" (at 477.52 64.77 0) (effects (font (size 1 1)) (hide yes)))
@@
                   (in_bom yes) (on_board yes) (dnp no)
                   (property "Reference" "C602" (at 208.28 99.13999999999999 0) (effects (font (size 1.27 1.27))))
-                  (property "Value" "100n 16V" (at 208.28 101.63999999999999 0) (effects (font (size 1.0 1.0))))
+                  (property "Value" "100n 50V" (at 208.28 101.63999999999999 0) (effects (font (size 1.0 1.0))))
                   (property "Footprint" "Capacitor_SMD:C_0603_1608Metric" (at 208.28 111.75999999999999 0) (effects (font (size 1 1)) (hide yes)))
                   (property "Datasheet" "https://www.yageogroup.com/component-documentation/download/specsheet/CC0603KRX7R9BB104" (at 208.28 111.75999999999999 0) (effects (font (size 1 1)) (hide yes)))
