File: hardware/pcb/kino-d4-carrier-a0/08_sensors.kicad_sch (KiCad schematic)
At the start: 9 parts, among them J800 3V PRIMARY RTC BACKUP, U800 LSM6DSOXTR, U801 RV-3028-C7, U802 TMP117AIDRVR

Commit message: feat(hardware): carrier A0.2 release pass - ready for fabrication with manual checks
Release review of the routed A0.2 carrier (A02-RELEASE.md: release matrix,
manual checks before ordering, bring-up tests). Final status: READY FOR
FABRICATION WITH SPECIFIC MANUAL CHECKS.

- USB-C input survives an unprogrammed STUSB4500 (20 V): D1001 SMF22A,
  R1004 10k, PD and load-switch P-FETs AO4409.
- Boost enable: R1204 100k BOOST_ENABLE to SYS_RAW (LTC2955-1 EN is a 2 uA
  source), Q1202 PMV16UN.
- I2C buffer U100 sides swapped (local bus on the TCA9517 A side's hard
  low); R100/R101 2.2k/22k hold EN low with JP1 pin 1 open.
- R105 SYNC_MASTER pull-down; D903 ESD on FN_N; TP1001 removed.
- SYS_RAW battery path as B.Cu and In2 pours with 25 extra vias; 1 oz inner
  copper in the stackup.
- XIAO socket pads get their solder-mask openings (footprint generator bug).
- Three fiducials per face; vias out of and away from pads; U1200 outline and
  pin-1 mark; legend lines and strokes 0.15 mm; silk association pass;
  CARRIER A0.2 / 2026-10 / S/N marking.
- Fab package (fab_a02.py): Gerbers + job file, drill, zip, placement files,
  fab BOM matched to LCSC by part number, hand-fit socket list, fab notes.
- Firmware constants header kino_carrier_a02.h.

DRC 0 / unconnected 0, ERC 0, verify.py --a02 passes.

Co-Authored-By: Claude Opus 5.5 <noreply@anthropic.com>
Parts:
- C800, C801, C802, C803: value 100n 16V -> 100n 50V
Other:
- note added: "IMU mode 1; axes follow the LSM6DSOX pin-1 orientation (not marked on silk). RTC backup charging must stay disabled for primary cell. No always-on wake promise."
- note removed: "IMU mode 1; axes marked on PCB. RTC backup charging must stay disabled for primary cell. No always-on wake promise."
Changed lines of the file:
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@@
       (company "KINO") (comment 1 "ENGINEERING DRAFT - NOT FOR FABRICATION"))
 (text "Motion, clock and board temperature" (at 15 12 0) (effects (font (size 2.5 2.5)) (justify left top)))
-(text "IMU mode 1; axes marked on PCB. RTC backup charging must stay disabled for primary cell. No always-on wake promise." (at 15 20 0) (effects (font (size 1.05 1.05)) (justify left top)))
+(text "IMU mode 1; axes follow the LSM6DSOX pin-1 orientation (not marked on silk). RTC backup charging must stay disabled for primary cell. No always-on wake promise." (at 15 20 0) (effects (font (size 1.05 1.05)) (justify left top)))
 (symbol (lib_id "KINO_A0:U800") (at 73.66 58.42 0) (unit 1)
                   (in_bom yes) (on_board yes) (dnp no)
@@
                   (in_bom yes) (on_board yes) (dnp no)
                   (property "Reference" "C800" (at 208.28 45.800000000000004 0) (effects (font (size 1.27 1.27))))
-                  (property "Value" "100n 16V" (at 208.28 48.300000000000004 0) (effects (font (size 1.0 1.0))))
+                  (property "Value" "100n 50V" (at 208.28 48.300000000000004 0) (effects (font (size 1.0 1.0))))
                   (property "Footprint" "Capacitor_SMD:C_0603_1608Metric" (at 208.28 58.42 0) (effects (font (size 1 1)) (hide yes)))
                   (property "Datasheet" "https://www.yageogroup.com/component-documentation/download/specsheet/CC0603KRX7R9BB104" (at 208.28 58.42 0) (effects (font (size 1 1)) (hide yes)))
@@
                   (in_bom yes) (on_board yes) (dnp no)
                   (property "Reference" "C801" (at 342.9 45.800000000000004 0) (effects (font (size 1.27 1.27))))
-                  (property "Value" "100n 16V" (at 342.9 48.300000000000004 0) (effects (font (size 1.0 1.0))))
+                  (property "Value" "100n 50V" (at 342.9 48.300000000000004 0) (effects (font (size 1.0 1.0))))
                   (property "Footprint" "Capacitor_SMD:C_0603_1608Metric" (at 342.9 58.42 0) (effects (font (size 1 1)) (hide yes)))
                   (property "Datasheet" "https://www.yageogroup.com/component-documentation/download/specsheet/CC0603KRX7R9BB104" (at 342.9 58.42 0) (effects (font (size 1 1)) (hide yes)))
@@
                   (in_bom yes) (on_board yes) (dnp no)
                   (property "Reference" "C802" (at 73.66 83.9 0) (effects (font (size 1.27 1.27))))
-                  (property "Value" "100n 16V" (at 73.66 86.4 0) (effects (font (size 1.0 1.0))))
+                  (property "Value" "100n 50V" (at 73.66 86.4 0) (effects (font (size 1.0 1.0))))
                   (property "Footprint" "Capacitor_SMD:C_0603_1608Metric" (at 73.66 96.52000000000001 0) (effects (font (size 1 1)) (hide yes)))
                   (property "Datasheet" "https://www.yageogroup.com/component-documentation/download/specsheet/CC0603KRX7R9BB104" (at 73.66 96.52000000000001 0) (effects (font (size 1 1)) (hide yes)))
@@
                   (in_bom yes) (on_board yes) (dnp no)
                   (property "Reference" "C803" (at 73.66 119.45999999999998 0) (effects (font (size 1.27 1.27))))
-                  (property "Value" "100n 16V" (at 73.66 121.95999999999998 0) (effects (font (size 1.0 1.0))))
+                  (property "Value" "100n 50V" (at 73.66 121.95999999999998 0) (effects (font (size 1.0 1.0))))
                   (property "Footprint" "Capacitor_SMD:C_0603_1608Metric" (at 73.66 132.07999999999998 0) (effects (font (size 1 1)) (hide yes)))
                   (property "Datasheet" "https://www.yageogroup.com/component-documentation/download/specsheet/CC0603KRX7R9BB104" (at 73.66 132.07999999999998 0) (effects (font (size 1 1)) (hide yes)))
