File: hardware/pcb/kino-d4-carrier-a0/10_usb_pd.kicad_sch (KiCad schematic)
At the start: 18 parts, among them J1000 USB4105-GF-A, Q1000 AO4407A, Q1001 AO4407A, U1000 STUSB4500QTR

Commit message: feat(hardware): carrier A0.2 release pass - ready for fabrication with manual checks
Release review of the routed A0.2 carrier (A02-RELEASE.md: release matrix,
manual checks before ordering, bring-up tests). Final status: READY FOR
FABRICATION WITH SPECIFIC MANUAL CHECKS.

- USB-C input survives an unprogrammed STUSB4500 (20 V): D1001 SMF22A,
  R1004 10k, PD and load-switch P-FETs AO4409.
- Boost enable: R1204 100k BOOST_ENABLE to SYS_RAW (LTC2955-1 EN is a 2 uA
  source), Q1202 PMV16UN.
- I2C buffer U100 sides swapped (local bus on the TCA9517 A side's hard
  low); R100/R101 2.2k/22k hold EN low with JP1 pin 1 open.
- R105 SYNC_MASTER pull-down; D903 ESD on FN_N; TP1001 removed.
- SYS_RAW battery path as B.Cu and In2 pours with 25 extra vias; 1 oz inner
  copper in the stackup.
- XIAO socket pads get their solder-mask openings (footprint generator bug).
- Three fiducials per face; vias out of and away from pads; U1200 outline and
  pin-1 mark; legend lines and strokes 0.15 mm; silk association pass;
  CARRIER A0.2 / 2026-10 / S/N marking.
- Fab package (fab_a02.py): Gerbers + job file, drill, zip, placement files,
  fab BOM matched to LCSC by part number, hand-fit socket list, fab notes.
- Firmware constants header kino_carrier_a02.h.

DRC 0 / unconnected 0, ERC 0, verify.py --a02 passes.

Co-Authored-By: Claude Opus 5.5 <noreply@anthropic.com>
Parts:
- removed TP1001: PD_9V_OK_N, TestPoint:TestPoint_Pad_D1.5mm, symbol KINO_A0:TP1001
- C1000: value 1u 35V -> 1u 50V
- D1001: value SMF12A -> SMF22A; Design note (none) -> VRWM 22 V: no conduction on a 20 V contract (unprogrammed S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
- Q1000, Q1001: value AO4407A -> AO4409; Design note Verify exact AO4407A manufacturer and SO8 pinout before BOM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 -> AO4409, SO-8: S pins 1-3, G pin 4, D pins 5-8. VDS -30 V, V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
- R1004: value 1k -> 10k; Design note (none) -> Above 10 V VBUS D1000 conducts through this resistor: 1.2 m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
Connections:
- net PD_9V_OK_N: no longer names the net of U1000.20 (POWER_OK2)
- no-connect marks 12 -> 13
Other:
- note added: "Charge-only port. Safe with the factory NVM (5/15/20 V PDOs, highest taken): TVS, FETs, gate network and charger are rated for a 20 V contract. Program the STUSB4500 NVM for 9V/2A with 5V fallback for normal use. Hot-plug transient at 20 V to be measured."
- note removed: "Charge-only port. STUSB4500 NVM must be programmed for 5V fallback and 9V/2A. Protection and gate transient review OPEN."
Changed lines of the file:
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@@
       (company "KINO") (comment 1 "ENGINEERING DRAFT - NOT FOR FABRICATION"))
 (text "USB-C PD sink and protected input" (at 15 12 0) (effects (font (size 2.5 2.5)) (justify left top)))
-(text "Charge-only port. STUSB4500 NVM must be programmed for 5V fallback and 9V/2A. Protection and gate transient review OPEN." (at 15 20 0) (effects (font (size 1.05 1.05)) (justify left top)))
+(text "Charge-only port. Safe with the factory NVM (5/15/20 V PDOs, highest taken): TVS, FETs, gate network and charger are rated for a 20 V contract. Program the STUSB4500 NVM for 9V/2A with 5V fallback for normal use. Hot-plug transient at 20 V to be measured." (at 15 20 0) (effects (font (size 1.05 1.05)) (justify left top)))
 (symbol (lib_id "KINO_A0:J1000") (at 73.66 66.03999999999999 0) (unit 1)
                   (in_bom yes) (on_board yes) (dnp no)
@@
                     (property "Intersheetrefs" "${INTERSHEET_REFS}" (at 231.14000000000001 60.959999999999994 180) (effects (font (size 0.8 0.8)) (hide yes))))
 (no_connect (at 226.06 63.499999999999986))
-(wire (pts (xy 226.06 66.03999999999999) (xy 231.14000000000001 66.03999999999999)) (stroke (width 0) (type default)))
-(global_label "PD_9V_OK_N" (shape bidirectional) (at 231.14000000000001 66.03999999999999 180)
-                    (effects (font (size 0.9 0.9)) (justify left))
-                    (property "Intersheetrefs" "${INTERSHEET_REFS}" (at 231.14000000000001 66.03999999999999 180) (effects (font (size 0.8 0.8)) (hide yes))))
+(no_connect (at 226.06 66.03999999999999))
 (wire (pts (xy 226.06 68.57999999999998) (xy 231.14000000000001 68.57999999999998)) (stroke (width 0) (type default)))
 (global_label "PD_1V2" (shape bidirectional) (at 231.14000000000001 68.57999999999998 180)
@@
                   (in_bom yes) (on_board yes) (dnp no)
                   (property "Reference" "C1000" (at 342.9 53.419999999999995 0) (effects (font (size 1.27 1.27))))
-                  (property "Value" "1u 35V" (at 342.9 55.919999999999995 0) (effects (font (size 1.0 1.0))))
+                  (property "Value" "1u 50V" (at 342.9 55.919999999999995 0) (effects (font (size 1.0 1.0))))
                   (property "Footprint" "Capacitor_SMD:C_0805_2012Metric" (at 342.9 66.03999999999999 0) (effects (font (size 1 1)) (hide yes)))
                   (property "Datasheet" "https://weblib.samsungsem.com/mlcc/mlcc-ec-data-sheet.do?partNumber=CL21B105KBFNNN" (at 342.9 66.03999999999999 0) (effects (font (size 1 1)) (hide yes)))
@@
                   (in_bom yes) (on_board yes) (dnp no)
                   (property "Reference" "Q1000" (at 73.66 135.97 0) (effects (font (size 1.27 1.27))))
-                  (property "Value" "AO4407A" (at 73.66 138.47 0) (effects (font (size 1.0 1.0))))
+                  (property "Value" "AO4409" (at 73.66 138.47 0) (effects (font (size 1.0 1.0))))
                   (property "Footprint" "Package_SO:SOIC-8_3.9x4.9mm_P1.27mm" (at 73.66 147.32 0) (effects (font (size 1 1)) (hide yes)))
-                  (property "Datasheet" "https://www.aosmd.com/sites/default/files/res/datasheets/AO4407A.pdf" (at 73.66 147.32 0) (effects (font (size 1 1)) (hide yes)))
-                  (property "Design note" "Verify exact AO4407A manufacturer and SO8 pinout before BOM release." (at 73.66 147.32 0) (effects (font (size 1 1)) (hide yes)))
+                  (property "Datasheet" "https://aosmd.com/sites/default/files/res/datasheets/AO4409.pdf" (at 73.66 147.32 0) (effects (font (size 1 1)) (hide yes)))
+                  (property "Design note" "AO4409, SO-8: S pins 1-3, G pin 4, D pins 5-8. VDS -30 V, VGS +/-20 V, RDS(on) 12 mOhm max at -4.5 V (the 5 V gate drive here). Replaces AO4407A, which is specified only down to -6 V." (at 73.66 147.32 0) (effects (font (size 1 1)) (hide yes)))
                   (pin "1")(pin "2")(pin "3")(pin "4")(pin "5")(pin "6")(pin "7")(pin "8")
                   (instances (project "KINO_D4_Carrier_A0" (path "/3e6ce248-02da-5043-9ed8-b7ca2a49de29/5aa1220a-e17d-547d-8acf-276839514db8" (reference "Q1000") (unit 1)))))
@@
                   (in_bom yes) (on_board yes) (dnp no)
                   (property "Reference" "Q1001" (at 208.28 135.97 0) (effects (font (size 1.27 1.27))))
-                  (property "Value" "AO4407A" (at 208.28 138.47 0) (effects (font (size 1.0 1.0))))
+                  (property "Value" "AO4409" (at 208.28 138.47 0) (effects (font (size 1.0 1.0))))
                   (property "Footprint" "Package_SO:SOIC-8_3.9x4.9mm_P1.27mm" (at 208.28 147.32 0) (effects (font (size 1 1)) (hide yes)))
-                  (property "Datasheet" "https://www.aosmd.com/sites/default/files/res/datasheets/AO4407A.pdf" (at 208.28 147.32 0) (effects (font (size 1 1)) (hide yes)))
-                  (property "Design note" "Verify exact AO4407A manufacturer and SO8 pinout before BOM release." (at 208.28 147.32 0) (effects (font (size 1 1)) (hide yes)))
+                  (property "Datasheet" "https://aosmd.com/sites/default/files/res/datasheets/AO4409.pdf" (at 208.28 147.32 0) (effects (font (size 1 1)) (hide yes)))
+                  (property "Design note" "AO4409, SO-8: S pins 1-3, G pin 4, D pins 5-8. VDS -30 V, VGS +/-20 V, RDS(on) 12 mOhm max at -4.5 V (the 5 V gate drive here). Replaces AO4407A, which is specified only down to -6 V." (at 208.28 147.32 0) (effects (font (size 1 1)) (hide yes)))
                   (pin "1")(pin "2")(pin "3")(pin "4")(pin "5")(pin "6")(pin "7")(pin "8")
                   (instances (project "KINO_D4_Carrier_A0" (path "/3e6ce248-02da-5043-9ed8-b7ca2a49de29/5aa1220a-e17d-547d-8acf-276839514db8" (reference "Q1001") (unit 1)))))
@@
                   (in_bom yes) (on_board yes) (dnp no)
                   (property "Reference" "R1004" (at 477.52 134.7 0) (effects (font (size 1.27 1.27))))
-                  (property "Value" "1k" (at 477.52 137.2 0) (effects (font (size 1.0 1.0))))
+                  (property "Value" "10k" (at 477.52 137.2 0) (effects (font (size 1.0 1.0))))
                   (property "Footprint" "Resistor_SMD:R_0603_1608Metric" (at 477.52 147.32 0) (effects (font (size 1 1)) (hide yes)))
-                  (property "Datasheet" "https://www.yageogroup.com/component-documentation/download/specsheet/RC0603FR-071KL" (at 477.52 147.32 0) (effects (font (size 1 1)) (hide yes)))
-                  (property "Design note" "" (at 477.52 147.32 0) (effects (font (size 1 1)) (hide yes)))
+                  (property "Datasheet" "https://www.yageogroup.com/component-documentation/download/specsheet/RC0603FR-0710KL" (at 477.52 147.32 0) (effects (font (size 1 1)) (hide yes)))
+                  (property "Design note" "Above 10 V VBUS D1000 conducts through this resistor: 1.2 mA at 22 V, inside the 3 mA VBUS_EN_SNK test condition (ST reference: 22k). Gate at -4.55 V at 5 V VBUS." (at 477.52 147.32 0) (effects (font (size 1 1)) (hide yes)))
                   (pin "1")(pin "2")
                   (instances (project "KINO_D4_Carrier_A0" (path "/3e6ce248-02da-5043-9ed8-b7ca2a49de29/5aa1220a-e17d-547d-8acf-276839514db8" (reference "R1004") (unit 1)))))
@@
                   (in_bom yes) (on_board yes) (dnp no)
                   (property "Reference" "D1001" (at 208.28 170.26 0) (effects (font (size 1.27 1.27))))
-                  (property "Value" "SMF12A" (at 208.28 172.76 0) (effects (font (size 1.0 1.0))))
+                  (property "Value" "SMF22A" (at 208.28 172.76 0) (effects (font (size 1.0 1.0))))
                   (property "Footprint" "Diode_SMD:D_SOD-123F" (at 208.28 182.88 0) (effects (font (size 1 1)) (hide yes)))
                   (property "Datasheet" "https://www.vishay.com/docs/85881/smf5v0atosmf58a.pdf" (at 208.28 182.88 0) (effects (font (size 1 1)) (hide yes)))
-                  (property "Design note" "" (at 208.28 182.88 0) (effects (font (size 1 1)) (hide yes)))
+                  (property "Design note" "VRWM 22 V: no conduction on a 20 V contract (unprogrammed STUSB4500 NVM). VBR 24.4-27 V, under the 28 V STUSB4500 and 30 V charger/FET ratings at low current." (at 208.28 182.88 0) (effects (font (size 1 1)) (hide yes)))
                   (pin "1")(pin "2")
                   (instances (project "KINO_D4_Carrier_A0" (path "/3e6ce248-02da-5043-9ed8-b7ca2a49de29/5aa1220a-e17d-547d-8acf-276839514db8" (reference "D1001") (unit 1)))))
@@
                     (effects (font (size 0.9 0.9)) (justify right))
                     (property "Intersheetrefs" "${INTERSHEET_REFS}" (at 60.959999999999994 215.9 0) (effects (font (size 0.8 0.8)) (hide yes))))
-(symbol (lib_id "KINO_A0:TP1001") (at 208.28 215.9 0) (unit 1)
-                  (in_bom yes) (on_board yes) (dnp no)
-                  (property "Reference" "TP1001" (at 208.28 205.82 0) (effects (font (size 1.27 1.27))))
-                  (property "Value" "PD_9V_OK_N" (at 208.28 208.32 0) (effects (font (size 1.0 1.0))))
-                  (property "Footprint" "TestPoint:TestPoint_Pad_D1.5mm" (at 208.28 215.9 0) (effects (font (size 1 1)) (hide yes)))
-                  (property "Datasheet" "" (at 208.28 215.9 0) (effects (font (size 1 1)) (hide yes)))
-                  (property "Design note" "" (at 208.28 215.9 0) (effects (font (size 1 1)) (hide yes)))
-                  (pin "1")
-                  (instances (project "KINO_D4_Carrier_A0" (path "/3e6ce248-02da-5043-9ed8-b7ca2a49de29/5aa1220a-e17d-547d-8acf-276839514db8" (reference "TP1001") (unit 1)))))
-(wire (pts (xy 200.66 215.9) (xy 195.57999999999998 215.9)) (stroke (width 0) (type default)))
-(global_label "PD_9V_OK_N" (shape bidirectional) (at 195.57999999999998 215.9 0)
-                    (effects (font (size 0.9 0.9)) (justify right))
-                    (property "Intersheetrefs" "${INTERSHEET_REFS}" (at 195.57999999999998 215.9 0) (effects (font (size 0.8 0.8)) (hide yes))))
 (embedded_fonts no))
