File: hardware/pcb/kino-d4-carrier-a0/11_charger.kicad_sch (KiCad schematic)
At the start: 36 parts, among them J1100 PROTECTED 1S PACK / NTC, U1100 BQ25798RQMR

Commit message: feat(hardware): carrier A0.2 - power-side opens, power-button corner
- MB_3V3: three router links join the U900 group, R902 and the main rail.
- Gauge (U701): R701 (BIN pull-down) moves beside its pin, and R702 (GPOUT
  pull-up) moves to the board edge.
- PD controller (U1000): R1004 moves above pin 16, PD_VBUS_SENSE loops
  round it, and C1000 moves onto the USB_VBUS run.
- STAT and charge LED: the charger STAT pin has no layout path out of its
  power copper. It is left open, firmware reads the charge state over I2C,
  and the expander STAT input goes. D1301 (charge LED), R1304, R1109 and
  TP1100 leave the design.
- Power LED: R1303 and D1300 move below U1300.
- Power controller (U1300): C1301 moves beside pin 3. PB and EN drop
  through new vias, and EN runs along the bottom edge to Q1202.

DRC: no clearance or short errors, parity clean, ERC 0, 16 open
connections.

Co-Authored-By: Claude Opus 5.5 <noreply@anthropic.com>
Parts:
- removed R1109: 10k, Resistor_SMD:R_0603_1608Metric, symbol KINO_A0:R1109
- removed TP1100: CHARGE_STAT_N, TestPoint:TestPoint_Pad_D1.5mm, symbol KINO_A0:TP1100
Connections:
- net CHARGE_STAT_N: no longer names the net of U1100.1 (STAT)
- no-connect marks 4 -> 5
Other:
- note added: "CE pulled LOW: charges with the camera off, POR defaults 4.2 V / 1 A (PROG 3.00k, TI tables 7-1/7-2). 103AT-2 pack NTC, TS window 1-60 C (TI RT1 5.24k / RT2 30.31k). Open or shorted NTC suspends charge. Fit R1110 only to inhibit charging at bring-up. STAT (pin 1) is left open: the pin sits inside the charger power copper with no layout path out; firmware reads the charge state from the status reg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"
- note removed: "CE pulled LOW: charges with the camera off, POR defaults 4.2 V / 1 A (PROG 3.00k, TI tables 7-1/7-2). 103AT-2 pack NTC, TS window 1-60 C (TI RT1 5.24k / RT2 30.31k). Open or shorted NTC suspends charge. Fit R1110 only to inhibit charging at bring-up."
- moved on the sheet: TP1101
Changed lines of the file:
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@@
       (company "KINO") (comment 1 "ENGINEERING DRAFT - NOT FOR FABRICATION"))
 (text "1S charger and battery entry" (at 15 12 0) (effects (font (size 2.5 2.5)) (justify left top)))
-(text "CE pulled LOW: charges with the camera off, POR defaults 4.2 V / 1 A (PROG 3.00k, TI tables 7-1/7-2). 103AT-2 pack NTC, TS window 1-60 C (TI RT1 5.24k / RT2 30.31k). Open or shorted NTC suspends charge. Fit R1110 only to inhibit charging at bring-up." (at 15 20 0) (effects (font (size 1.05 1.05)) (justify left top)))
+(text "CE pulled LOW: charges with the camera off, POR defaults 4.2 V / 1 A (PROG 3.00k, TI tables 7-1/7-2). 103AT-2 pack NTC, TS window 1-60 C (TI RT1 5.24k / RT2 30.31k). Open or shorted NTC suspends charge. Fit R1110 only to inhibit charging at bring-up. STAT (pin 1) is left open: the pin sits inside the charger power copper with no layout path out; firmware reads the charge state from the status registers over I2C." (at 15 20 0) (effects (font (size 1.05 1.05)) (justify left top)))
 (symbol (lib_id "KINO_A0:J1100") (at 73.66 68.58 0) (unit 1)
                   (in_bom yes) (on_board yes) (dnp no)
@@
                   (pin "1")(pin "2")(pin "3")(pin "4")(pin "5")(pin "6")(pin "7")(pin "8")(pin "9")(pin "10")(pin "11")(pin "12")(pin "13")(pin "14")(pin "15")(pin "16")(pin "17")(pin "18")(pin "19")(pin "20")(pin "21")(pin "22")(pin "23")(pin "24")(pin "25")(pin "26")(pin "27")(pin "28")(pin "29")
                   (instances (project "KINO_D4_Carrier_A0" (path "/3e6ce248-02da-5043-9ed8-b7ca2a49de29/7db3d43e-d2ec-5c9b-9d22-bda4d57a7a9a" (reference "U1100") (unit 1)))))
-(wire (pts (xy 325.12 50.8) (xy 320.04 50.8)) (stroke (width 0) (type default)))
-(global_label "CHARGE_STAT_N" (shape bidirectional) (at 320.04 50.8 0)
-                    (effects (font (size 0.9 0.9)) (justify right))
-                    (property "Intersheetrefs" "${INTERSHEET_REFS}" (at 320.04 50.8 0) (effects (font (size 0.8 0.8)) (hide yes))))
+(no_connect (at 325.12 50.8))
 (wire (pts (xy 325.12 53.339999999999996) (xy 320.04 53.339999999999996)) (stroke (width 0) (type default)))
 (global_label "CHG_VBUS" (shape bidirectional) (at 320.04 53.339999999999996 0)
@@
                     (effects (font (size 0.9 0.9)) (justify left))
                     (property "Intersheetrefs" "${INTERSHEET_REFS}" (at 86.36 365.76 180) (effects (font (size 0.8 0.8)) (hide yes))))
-(symbol (lib_id "KINO_A0:R1109") (at 208.28 365.76 0) (unit 1)
-                  (in_bom yes) (on_board yes) (dnp no)
-                  (property "Reference" "R1109" (at 208.28 353.14 0) (effects (font (size 1.27 1.27))))
-                  (property "Value" "10k" (at 208.28 355.64 0) (effects (font (size 1.0 1.0))))
-                  (property "Footprint" "Resistor_SMD:R_0603_1608Metric" (at 208.28 365.76 0) (effects (font (size 1 1)) (hide yes)))
-                  (property "Datasheet" "https://www.yageogroup.com/component-documentation/download/specsheet/RC0603FR-0710KL" (at 208.28 365.76 0) (effects (font (size 1 1)) (hide yes)))
+(symbol (lib_id "KINO_A0:TP1101") (at 208.28 365.76 0) (unit 1)
+                  (in_bom yes) (on_board yes) (dnp no)
+                  (property "Reference" "TP1101" (at 208.28 355.68 0) (effects (font (size 1.27 1.27))))
+                  (property "Value" "SYS_RAW" (at 208.28 358.18 0) (effects (font (size 1.0 1.0))))
+                  (property "Footprint" "TestPoint:TestPoint_Pad_D1.5mm" (at 208.28 365.76 0) (effects (font (size 1 1)) (hide yes)))
+                  (property "Datasheet" "" (at 208.28 365.76 0) (effects (font (size 1 1)) (hide yes)))
                   (property "Design note" "" (at 208.28 365.76 0) (effects (font (size 1 1)) (hide yes)))
-                  (pin "1")(pin "2")
-                  (instances (project "KINO_D4_Carrier_A0" (path "/3e6ce248-02da-5043-9ed8-b7ca2a49de29/7db3d43e-d2ec-5c9b-9d22-bda4d57a7a9a" (reference "R1109") (unit 1)))))
-(wire (pts (xy 200.66 365.76) (xy 195.57999999999998 365.76)) (stroke (width 0) (type default)))
-(global_label "CHARGE_STAT_N" (shape bidirectional) (at 195.57999999999998 365.76 0)
-                    (effects (font (size 0.9 0.9)) (justify right))
-                    (property "Intersheetrefs" "${INTERSHEET_REFS}" (at 195.57999999999998 365.76 0) (effects (font (size 0.8 0.8)) (hide yes))))
-(wire (pts (xy 215.9 365.76) (xy 220.98000000000002 365.76)) (stroke (width 0) (type default)))
-(global_label "MB_3V3" (shape bidirectional) (at 220.98000000000002 365.76 180)
-                    (effects (font (size 0.9 0.9)) (justify left))
-                    (property "Intersheetrefs" "${INTERSHEET_REFS}" (at 220.98000000000002 365.76 180) (effects (font (size 0.8 0.8)) (hide yes))))
-(symbol (lib_id "KINO_A0:TP1100") (at 342.9 365.76 0) (unit 1)
-                  (in_bom yes) (on_board yes) (dnp no)
-                  (property "Reference" "TP1100" (at 342.9 355.68 0) (effects (font (size 1.27 1.27))))
-                  (property "Value" "CHARGE_STAT_N" (at 342.9 358.18 0) (effects (font (size 1.0 1.0))))
-                  (property "Footprint" "TestPoint:TestPoint_Pad_D1.5mm" (at 342.9 365.76 0) (effects (font (size 1 1)) (hide yes)))
-                  (property "Datasheet" "" (at 342.9 365.76 0) (effects (font (size 1 1)) (hide yes)))
-                  (property "Design note" "" (at 342.9 365.76 0) (effects (font (size 1 1)) (hide yes)))
-                  (pin "1")
-                  (instances (project "KINO_D4_Carrier_A0" (path "/3e6ce248-02da-5043-9ed8-b7ca2a49de29/7db3d43e-d2ec-5c9b-9d22-bda4d57a7a9a" (reference "TP1100") (unit 1)))))
-(wire (pts (xy 335.28 365.76) (xy 330.2 365.76)) (stroke (width 0) (type default)))
-(global_label "CHARGE_STAT_N" (shape bidirectional) (at 330.2 365.76 0)
-                    (effects (font (size 0.9 0.9)) (justify right))
-                    (property "Intersheetrefs" "${INTERSHEET_REFS}" (at 330.2 365.76 0) (effects (font (size 0.8 0.8)) (hide yes))))
-(symbol (lib_id "KINO_A0:TP1101") (at 477.52 365.76 0) (unit 1)
-                  (in_bom yes) (on_board yes) (dnp no)
-                  (property "Reference" "TP1101" (at 477.52 355.68 0) (effects (font (size 1.27 1.27))))
-                  (property "Value" "SYS_RAW" (at 477.52 358.18 0) (effects (font (size 1.0 1.0))))
-                  (property "Footprint" "TestPoint:TestPoint_Pad_D1.5mm" (at 477.52 365.76 0) (effects (font (size 1 1)) (hide yes)))
-                  (property "Datasheet" "" (at 477.52 365.76 0) (effects (font (size 1 1)) (hide yes)))
-                  (property "Design note" "" (at 477.52 365.76 0) (effects (font (size 1 1)) (hide yes)))
                   (pin "1")
                   (instances (project "KINO_D4_Carrier_A0" (path "/3e6ce248-02da-5043-9ed8-b7ca2a49de29/7db3d43e-d2ec-5c9b-9d22-bda4d57a7a9a" (reference "TP1101") (unit 1)))))
-(wire (pts (xy 469.9 365.76) (xy 464.82 365.76)) (stroke (width 0) (type default)))
-(global_label "SYS_RAW" (shape bidirectional) (at 464.82 365.76 0)
-                    (effects (font (size 0.9 0.9)) (justify right))
-                    (property "Intersheetrefs" "${INTERSHEET_REFS}" (at 464.82 365.76 0) (effects (font (size 0.8 0.8)) (hide yes))))
+(wire (pts (xy 200.66 365.76) (xy 195.57999999999998 365.76)) (stroke (width 0) (type default)))
+(global_label "SYS_RAW" (shape bidirectional) (at 195.57999999999998 365.76 0)
+                    (effects (font (size 0.9 0.9)) (justify right))
+                    (property "Intersheetrefs" "${INTERSHEET_REFS}" (at 195.57999999999998 365.76 0) (effects (font (size 0.8 0.8)) (hide yes))))
 (embedded_fonts no))

Commit message: feat(hardware): carrier A0.2 release pass - ready for fabrication with manual checks
Release review of the routed A0.2 carrier (A02-RELEASE.md: release matrix,
manual checks before ordering, bring-up tests). Final status: READY FOR
FABRICATION WITH SPECIFIC MANUAL CHECKS.

- USB-C input survives an unprogrammed STUSB4500 (20 V): D1001 SMF22A,
  R1004 10k, PD and load-switch P-FETs AO4409.
- Boost enable: R1204 100k BOOST_ENABLE to SYS_RAW (LTC2955-1 EN is a 2 uA
  source), Q1202 PMV16UN.
- I2C buffer U100 sides swapped (local bus on the TCA9517 A side's hard
  low); R100/R101 2.2k/22k hold EN low with JP1 pin 1 open.
- R105 SYNC_MASTER pull-down; D903 ESD on FN_N; TP1001 removed.
- SYS_RAW battery path as B.Cu and In2 pours with 25 extra vias; 1 oz inner
  copper in the stackup.
- XIAO socket pads get their solder-mask openings (footprint generator bug).
- Three fiducials per face; vias out of and away from pads; U1200 outline and
  pin-1 mark; legend lines and strokes 0.15 mm; silk association pass;
  CARRIER A0.2 / 2026-10 / S/N marking.
- Fab package (fab_a02.py): Gerbers + job file, drill, zip, placement files,
  fab BOM matched to LCSC by part number, hand-fit socket list, fab notes.
- Firmware constants header kino_carrier_a02.h.

DRC 0 / unconnected 0, ERC 0, verify.py --a02 passes.

Co-Authored-By: Claude Opus 5.5 <noreply@anthropic.com>
Parts:
- C1104, C1105, C1107, C1108, C1109, C1111, C1112, C1113, C1114, C1115, C1117, C1118: value 10u 35V X7R -> 10u 50V X7R
- C1106, C1110, C1116, C1119: value 100n 35V -> 100n 50V
- R1100: Design note TI Table 7-1: 1S, 1.5MHz. Default 4.2V / 1A charge, hardwar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 -> TI Table 7-1: 1S, 1.5MHz. POR default 4.2 V / 1 A; charging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
- R1108: Design note NTC returns to pack negative = board GND; the gauge shunt i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 -> 0 ohm NTC link (bring-up): open it to measure the pack NTC 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
