File: hardware/pcb/kino-d4-carrier-a0/12_boost.kicad_sch (KiCad schematic)
At the start: 30 parts, among them Q1200 AO4407A, Q1201 AO4407A, Q1202 2N7002, U1200 TPS61288LRQQR, U1201 TPS62162DSGR

Commit message: feat(hardware): carrier A0.2 - external connections to the back, 0 ohm power links
- Cable connectors (J102, J601, J800, J900-J904, J1300), the camera GPIO
  breakout headers J201-J501, J101 and the P4 ribbon J100 move to B.Cu so
  the socketed XIAOs are the tallest parts on the front (MECHANICAL.md,
  face assignment). Pogo/sense contacts stay on the front.
- JP200-JP500 and JP1200 become Vishay CRCW12060000Z0EAHP 0 ohm links
  (10 A, <=5 mOhm) on a project land drawn from the Vishay reflow pads;
  capture, BOM, ERC and netlist regenerated.
- P4_5V_ISO feed re-run on In2 at 2.0 mm with 3-via layer changes.
- Connector labels follow their connectors to B.SilkS.
- 195 connections are open again after the move; DRC has no clearance,
  short, courtyard or silk errors (dangling lane ends only).

Co-Authored-By: Claude Opus 5.5 <noreply@anthropic.com>
Parts:
- JP1200: value REMOVE FOR P4 USB SERVICE -> 0R LINK - REMOVE FOR P4 USB SERVICE; footprint Connector_PinHeader_2.54mm:PinHeader_1x02_P2.54mm_Vertical -> KINO_A0:R_1206_3216Metric_Vishay_CRCW-HP; Design note Reverse isolation diode plus manual disconnect. Verify Guit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 -> Reverse isolation diode plus manual disconnect (0 ohm link,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
Changed lines of the file:
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@@
                   (in_bom yes) (on_board yes) (dnp no)
                   (property "Reference" "JP1200" (at 342.9 261.70000000000005 0) (effects (font (size 1.27 1.27))))
-                  (property "Value" "REMOVE FOR P4 USB SERVICE" (at 342.9 264.20000000000005 0) (effects (font (size 1.0 1.0))))
-                  (property "Footprint" "Connector_PinHeader_2.54mm:PinHeader_1x02_P2.54mm_Vertical" (at 342.9 271.78000000000003 0) (effects (font (size 1 1)) (hide yes)))
-                  (property "Datasheet" "https://www.we-online.com/components/products/datasheet/61300211121.pdf ; https://www.we-online.com/components/products/datasheet/60900213421.pdf" (at 342.9 271.78000000000003 0) (effects (font (size 1 1)) (hide yes)))
-                  (property "Design note" "Reverse isolation diode plus manual disconnect. Verify Guition external supply and USB topology before simultaneous connection." (at 342.9 271.78000000000003 0) (effects (font (size 1 1)) (hide yes)))
+                  (property "Value" "0R LINK - REMOVE FOR P4 USB SERVICE" (at 342.9 264.20000000000005 0) (effects (font (size 1.0 1.0))))
+                  (property "Footprint" "KINO_A0:R_1206_3216Metric_Vishay_CRCW-HP" (at 342.9 271.78000000000003 0) (effects (font (size 1 1)) (hide yes)))
+                  (property "Datasheet" "https://www.vishay.com/docs/20043/crcwhpe3.pdf" (at 342.9 271.78000000000003 0) (effects (font (size 1 1)) (hide yes)))
+                  (property "Design note" "Reverse isolation diode plus manual disconnect (0 ohm link, desolder for P4 USB service). Verify Guition external supply and USB topology before simultaneous connection." (at 342.9 271.78000000000003 0) (effects (font (size 1 1)) (hide yes)))
                   (pin "1")(pin "2")
                   (instances (project "KINO_D4_Carrier_A0" (path "/3e6ce248-02da-5043-9ed8-b7ca2a49de29/7b9b6bc4-2c97-56ef-abdc-8792495ea361" (reference "JP1200") (unit 1)))))

Commit message: feat(hardware): carrier A0.2 release pass - ready for fabrication with manual checks
Release review of the routed A0.2 carrier (A02-RELEASE.md: release matrix,
manual checks before ordering, bring-up tests). Final status: READY FOR
FABRICATION WITH SPECIFIC MANUAL CHECKS.

- USB-C input survives an unprogrammed STUSB4500 (20 V): D1001 SMF22A,
  R1004 10k, PD and load-switch P-FETs AO4409.
- Boost enable: R1204 100k BOOST_ENABLE to SYS_RAW (LTC2955-1 EN is a 2 uA
  source), Q1202 PMV16UN.
- I2C buffer U100 sides swapped (local bus on the TCA9517 A side's hard
  low); R100/R101 2.2k/22k hold EN low with JP1 pin 1 open.
- R105 SYNC_MASTER pull-down; D903 ESD on FN_N; TP1001 removed.
- SYS_RAW battery path as B.Cu and In2 pours with 25 extra vias; 1 oz inner
  copper in the stackup.
- XIAO socket pads get their solder-mask openings (footprint generator bug).
- Three fiducials per face; vias out of and away from pads; U1200 outline and
  pin-1 mark; legend lines and strokes 0.15 mm; silk association pass;
  CARRIER A0.2 / 2026-10 / S/N marking.
- Fab package (fab_a02.py): Gerbers + job file, drill, zip, placement files,
  fab BOM matched to LCSC by part number, hand-fit socket list, fab notes.
- Firmware constants header kino_carrier_a02.h.

DRC 0 / unconnected 0, ERC 0, verify.py --a02 passes.

Co-Authored-By: Claude Opus 5.5 <noreply@anthropic.com>
Parts:
- added R1204: 100k, Resistor_SMD:R_0603_1608Metric, symbol KINO_A0:R1204
- C1201: Design note (none) -> TPS61288 optional CP (TI eq 14). DNP; fit only if the bench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
- C1202: Design note TI: VCC needs > 1.0 uF effective; 2.2 uF 0603 is about 1.0 uF at 5 V. -> TI: VCC needs > 1.0 uF effective; 2.2 uF 0603 is about 1.0 uF at 5 V, hence 4.7 uF.
- C1205: value 100n 16V -> 100n 50V
- Q1200, Q1201: value AO4407A -> AO4409; Design note Verify exact AO4407A manufacturer and SO8 pinout before BOM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 -> AO4409, SO-8: S pins 1-3, G pin 4, D pins 5-8. VDS -30 V, V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
- Q1202: value 2N7002 -> PMV16UN; Design note (none) -> VGS(th) 0.4-1.0 V: fully on from BOOST_ENABLE at any SYS_RA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
Connections:
- net BOOST_ENABLE: now also R1204.1
- net SYS_RAW: now also R1204.2
Other:
- moved on the sheet: C1212, C1213, D1200, JP1200, L1201, TP1200, TP1201, TP1202, U1201
